Commit message: adding movement to urdf

File: modelos/irb120_3_58.urdf (robot description, URDF)
Before this commit: robot abb_irb120_3_58, 9 links, 8 joints
Links:
- link base_link: mass 6.215 -> None
- link link_1: mass 3.067 -> None
- link link_2: mass 3.909 -> None
- link link_3: mass 2.944 -> None
- link link_4: mass 1.328 -> None
- link link_5: mass 0.546 -> None
- link link_6: mass 0.137 -> None

File: modelos/irb5400.urdf (robot description, URDF)
Before this commit: robot abb_irb5400, 10 links, 9 joints
Joints:
- removed joint joint1
- removed joint joint2
- removed joint joint3
- removed joint joint4
- removed joint joint5
- removed joint joint6
- added joint joint_1: type revolute, parent base_link, child link_1, origin xyz=0 0 0 rpy=0 0 0, axis 0 0 1, limit lower=-2.617 upper=2.617 effort=100 velocity=2.3911
- added joint joint_2: type revolute, parent link_1, child link_2, origin xyz=0.300 0 0.660 rpy=0 0 0, axis 0 1 0, limit lower=-1.396 upper=1.396 effort=100 velocity=2.3911
- added joint joint_3: type revolute, parent link_2, child link_3, origin xyz=0 0 1.200 rpy=0 0 0, axis 0 1 0, limit lower=-1.308 upper=1.308 effort=100 velocity=2.3911
- added joint joint_4: type revolute, parent link_3, child link_4, origin xyz=1.339 0 0.186 rpy=0 0 0, axis 1 0 0, limit lower=-6.0 upper=6.0 effort=100 velocity=8.1157
- added joint joint_5: type revolute, parent link_4, child link_5, origin xyz=0.0693 0 0 rpy=0 0.6109 0, axis 1 0 0, limit lower=-6.0 upper=6.0 effort=100 velocity=6.1086
- added joint joint_6: type revolute, parent link_5b, child link_6, origin xyz=0.0672 0 -0.0470 rpy=0 0.6109 0, axis 1 0 0, limit lower=-6.0 upper=6.0 effort=100 velocity=9.3375

File: modelos/kr210l150.urdf (robot description, URDF)
Before this commit: robot kuka_kr210, 9 links, 8 joints
Joints:
- removed joint joint_a1
- removed joint joint_a2
- removed joint joint_a3
- removed joint joint_a4
- removed joint joint_a5
- removed joint joint_a6
- added joint joint_1: type revolute, parent base_link, child link_1, origin xyz=-0.00262 0.00097586 0.33099 rpy=0 0 0, axis 0 0 1, limit lower=-3.228859205 upper=3.228859205 effort=0 velocity=2.146755039
- added joint joint_2: type revolute, parent link_1, child link_2, origin xyz=0.35277 -0.037476 0.4192 rpy=0 0 0, axis 0 1 0, limit lower=-0.785398185 upper=1.483529905 effort=0 velocity=2.007128695
- added joint joint_3: type revolute, parent link_2, child link_3, origin xyz=-9.8483E-05 -0.1475 1.2499 rpy=0 0 0, axis 0 1 0, limit lower=-3.66519153 upper=1.134464045 effort=0 velocity=1.954768816
- added joint joint_4: type revolute, parent link_3, child link_4, origin xyz=0.95795 0.184 -0.055059 rpy=0 0 0, axis 1 0 0, limit lower=-6.10865255 upper=6.10865255 effort=0 velocity=3.124139447
- added joint joint_5: type revolute, parent link_4, child link_5, origin xyz=0.542 0 0 rpy=0 0 0, axis 0 1 0, limit lower=-2.181661625 upper=2.181661625 effort=0 velocity=3.001966396
- added joint joint_6: type revolute, parent link_5, child link_6, origin xyz=0.1925 0 0 rpy=0 0 0, axis 1 0 0, limit lower=-6.10865255 upper=6.10865255 effort=0 velocity=3.822271167

File: modelos/mh5.urdf (robot description, URDF)
Before this commit: robot motoman_mh5, 7 links, 6 joints
Joints:
- removed joint joint_b
- removed joint joint_l
- removed joint joint_r
- removed joint joint_s
- removed joint joint_t
- removed joint joint_u
- added joint joint_1: type revolute, parent base_link, child link_s, origin xyz=0 0 0.1990 rpy=0 0 0, axis 0 0 1, limit lower=-2.9671 upper=2.9671 effort=100 velocity=2.96
- added joint joint_2: type revolute, parent link_s, child link_l, origin xyz=0.0880 0 0.1310 rpy=0 0 0, axis 0 1 0, limit lower=-1.1345 upper=2.6180 effort=100 velocity=2.96
- added joint joint_3: type revolute, parent link_l, child link_u, origin xyz=0 0 0.3100 rpy=0 0 0, axis 0 -1 0, limit lower=-1.0122 upper=3.2218 effort=100 velocity=2.96
- added joint joint_4: type revolute, parent link_u, child link_r, origin xyz=0.0715 0 0.0399 rpy=0 0 0, axis -1 0 0, limit lower=-3.3161 upper=3.3161 effort=100 velocity=3.48
- added joint joint_5: type revolute, parent link_r, child link_b, origin xyz=0.2335 0 0 rpy=0 0 0, axis 0 -1 0, limit lower=-2.1817 upper=2.1817 effort=100 velocity=3.48
- added joint joint_6: type revolute, parent link_b, child link_t, origin xyz=0.0865 0 0 rpy=0 0 0, axis -1 0 0, limit lower=-6.2831 upper=6.2831 effort=100 velocity=6.97
