Commit message: Add delet param and param of robot TIP and ROOT URDF

File: modelos/mh5.urdf (robot description, URDF)
Before this commit: robot motoman_mh5, 7 links, 6 joints
Links:
- removed link link_b
- removed link link_l
- removed link link_r
- removed link link_s
- removed link link_t
- removed link link_u
- added link link_1; collision mesh filename=package://rvizglabre/modelos/mh5/collision/MH5_S_AXIS.stl; visual mesh filename=package://rvizglabre/modelos/mh5/visual/MH5_S_AXIS.stl
- added link link_2; collision mesh filename=package://rvizglabre/modelos/mh5/collision/MH5_L_AXIS.stl; visual mesh filename=package://rvizglabre/modelos/mh5/visual/MH5_L_AXIS.stl
- added link link_3; collision mesh filename=package://rvizglabre/modelos/mh5/collision/MH5_U_AXIS.stl; visual mesh filename=package://rvizglabre/modelos/mh5/visual/MH5_U_AXIS.stl
- added link link_4; collision mesh filename=package://rvizglabre/modelos/mh5/collision/MH5_R_AXIS.stl; visual mesh filename=package://rvizglabre/modelos/mh5/visual/MH5_R_AXIS.stl
- added link link_5; collision mesh filename=package://rvizglabre/modelos/mh5/collision/MH5_B_AXIS.stl; visual mesh filename=package://rvizglabre/modelos/mh5/visual/MH5_B_AXIS.stl
- added link link_6; collision mesh filename=package://rvizglabre/modelos/mh5/collision/MH5_T_AXIS.stl; visual mesh filename=package://rvizglabre/modelos/mh5/visual/MH5_T_AXIS.stl
Joints:
- joint joint_1: child link_s -> link_1
- joint joint_2: child link_l -> link_2; parent link_s -> link_1
- joint joint_3: child link_u -> link_3; parent link_l -> link_2
- joint joint_4: child link_r -> link_4; parent link_u -> link_3
- joint joint_5: child link_b -> link_5; parent link_r -> link_4
- joint joint_6: child link_t -> link_6; parent link_b -> link_5
