Commit message: corrected URDF FK

File: modelos/pan_tilt.urdf (robot description, URDF)
Before this commit: robot pan_tilt, 3 links, 2 joints
Links:
- removed link pan_link
- removed link tilt_link
- added link link_1, mass 1; collision cylinder length=0.4 radius=0.06; visual cylinder length=0.4 radius=0.04
- added link tool0, mass 1; collision cylinder length=0.4 radius=0.06; visual cylinder length=0.4 radius=0.04
Joints:
- removed joint pan_joint
- removed joint tilt_joint
- added joint joint_1: type revolute, parent base_link, child link_1, origin xyz=0 0 0.1, axis 0 0 1, limit lower=-3.14 upper=3.14 effort=300 velocity=0.1
- added joint joint_2: type revolute, parent link_1, child tool0, origin xyz=0 0 0.2, axis 0 1 0, limit lower=-4.64 upper=-1.5 effort=300 velocity=0.1
