Commit message: Cylindrical Robot

File: modelos/cylindrical.urdf (robot description, URDF)
Before this commit: robot Cylindrical, 2 links, 1 joints
Links:
- added link link_2; visual box size=0.06 0.7 0.08
- added link link_3; visual box size=0.05 0.4 0.05
- link base_link: geometry visual box size=1.0 1.0 0.05; visual cylinder length=0.05 radius=0.15
- link link_1: geometry visual cylinder length=1 radius=0.025
Joints:
- added joint joint_2: type prismatic, parent link_1, child link_2, origin xyz=0 0 0.075 rpy=0 0 0, axis 0 0 1, limit lower=0 upper=0.85 effort=1000.0 velocity=1.0
- added joint joint_3: type prismatic, parent link_2, child link_3, origin xyz=0 0.55 0 rpy=0 0 0, axis 0 1 0, limit lower=0 upper=0.35 effort=1000.0 velocity=1.0
- joint joint_1: origin xyz=0 0 0 rpy=0 0 0 -> xyz=0 0 0.05 rpy=0 0 0

Commit message: first test, joints with timer sleep

File: modelos/cylindrical.urdf (robot description, URDF)
Before this commit: robot Cylindrical, 4 links, 3 joints
Links:
- added link tool0
Joints:
- added joint joint3-tool0: type fixed, parent link_3, child tool0, origin xyz=0 0 0 rpy=0 0 0
