Commit message: Moveit robot display

File: modelos/3dof.urdf (robot description, URDF)
Before this commit: robot threeseg, 5 links, 4 joints
Joints:
- removed joint joint_4
- added joint joint_4-tool0: type revolute, parent link_3, child tool0, origin xyz=0 0 1 rpy=0 0 0, axis 0 0 1, limit lower=-6.28318 upper=6.28318 effort=30 velocity=1.0

Commit message: Case DH parameters

File: modelos/3dof.urdf (robot description, URDF)
Before this commit: robot threeseg, 5 links, 4 joints
Links:
- link link_1: geometry visual box size=0.1 0.1 1
- link link_2: geometry visual box size=0.1 0.1 0.5
- link link_3: geometry visual box size=0.1 0.1 0.5
Joints:
- joint joint_2: origin xyz=0 0 3 rpy=-0.785398 0 0 -> xyz=0 0 1 rpy=0 0 0
- joint joint_3: origin xyz=0 0 2 rpy=-0.5 0 0 -> xyz=0 0 0.5 rpy=0 0 0
- joint joint_4-tool0: origin xyz=0 0 1 rpy=0 0 0 -> xyz=0 0 0.5 rpy=0 0 0

File: modelos/two_link_yz.urdf (robot description, URDF)
Before this commit: robot 2dof, 4 links, 3 joints
Joints:
- joint joint_3: axis 0 0 1 -> 1 0 0
