Commit message: Dialer update to Value of Joint of URDF

File: modelos/kr16_2.urdf (robot description, URDF)
Before this commit: robot kuka_kr16_2, 9 links, 8 joints
Joints:
- removed joint joint_a1
- removed joint joint_a2
- removed joint joint_a3
- removed joint joint_a4
- removed joint joint_a5
- removed joint joint_a6
- added joint joint_1: type revolute, parent base_link, child link_1, origin xyz=0 0 0.675 rpy=0 0 0, axis 0 0 -1, limit lower=-3.22885911619 upper=3.22885911619 effort=0 velocity=2.72271363311
- added joint joint_2: type revolute, parent link_1, child link_2, origin xyz=0.26 0 0 rpy=0 0 0, axis 0 1 0, limit lower=-2.70526034059 upper=0.610865238198 effort=0 velocity=2.72271363311
- added joint joint_3: type revolute, parent link_2, child link_3, origin xyz=0.68 0 0 rpy=0 0 0, axis 0 1 0, limit lower=-2.26892802759 upper=2.68780704807 effort=0 velocity=2.72271363311
- added joint joint_4: type revolute, parent link_3, child link_4, origin xyz=0.67 0 -0.035 rpy=0 0 0, axis -1 0 0, limit lower=-6.10865238198 upper=6.10865238198 effort=0 velocity=5.75958653158
- added joint joint_5: type revolute, parent link_4, child link_5, origin xyz=0 0 0 rpy=0 0 0, axis 0 1 0, limit lower=-2.26892802759 upper=2.26892802759 effort=0 velocity=5.75958653158
- added joint joint_6: type revolute, parent link_5, child link_6, origin xyz=0 0 0 rpy=0 0 0, axis -1 0 0, limit lower=-6.10865238198 upper=6.10865238198 effort=0 velocity=10.7337748998

File: modelos/sia10f.urdf (robot description, URDF)
Before this commit: robot motoman_sia10f, 9 links, 8 joints
Links:
- removed link link_b
- removed link link_e
- removed link link_l
- removed link link_r
- removed link link_s
- removed link link_t
- removed link link_u
- added link link_1; collision mesh filename=package://rvizglabre/modelos/sia10f/collision/motoman_axis_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; visual mesh filename=package://rvizglabre/modelos/sia10f/visual/motoman_axis_s.s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
- added link link_2; collision mesh filename=package://rvizglabre/modelos/sia10f/collision/motoman_axis_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; visual mesh filename=package://rvizglabre/modelos/sia10f/visual/motoman_axis_l.s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
- added link link_3; collision mesh filename=package://rvizglabre/modelos/sia10f/collision/motoman_axis_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; visual mesh filename=package://rvizglabre/modelos/sia10f/visual/motoman_axis_e.s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
- added link link_4; collision mesh filename=package://rvizglabre/modelos/sia10f/collision/motoman_axis_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; visual mesh filename=package://rvizglabre/modelos/sia10f/visual/motoman_axis_u.s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
- added link link_5; collision mesh filename=package://rvizglabre/modelos/sia10f/collision/motoman_axis_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; visual mesh filename=package://rvizglabre/modelos/sia10f/visual/motoman_axis_r.s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
- added link link_6; collision mesh filename=package://rvizglabre/modelos/sia10f/collision/motoman_axis_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; visual mesh filename=package://rvizglabre/modelos/sia10f/visual/motoman_axis_b.s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
- added link link_7; collision mesh filename=package://rvizglabre/modelos/sia10f/collision/motoman_axis_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; visual mesh filename=package://rvizglabre/modelos/sia10f/visual/motoman_axis_t.s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
Joints:
- removed joint joint_b
- removed joint joint_e
- removed joint joint_l
- removed joint joint_r
- removed joint joint_s
- removed joint joint_t
- removed joint joint_u
- removed joint link_l-base
- added joint joint_1: type revolute, parent base_link, child link_1, origin xyz=0 0 0.36 rpy=0 0 0, axis 0 0 1, limit lower=-3.1415 upper=3.1415 effort=100 velocity=2.9670
- added joint joint_2: type revolute, parent link_1, child link_2, origin xyz=0 0 0 rpy=0 0 0, axis 0 1 0, limit lower=-1.9198 upper=1.9198 effort=100 velocity=2.9670
- added joint joint_3: type revolute, parent link_2, child link_3, origin xyz=0 0 0.36 rpy=0 0 0, axis 0 0 1, limit lower=-2.9670 upper=2.9670 effort=100 velocity=2.9670
- added joint joint_4: type revolute, parent link_3, child link_4, origin xyz=0 0 0 rpy=0 0 0, axis 0 -1 0, limit lower=-2.3561 upper=2.3561 effort=100 velocity=2.9670
- added joint joint_5: type revolute, parent link_4, child link_5, origin xyz=0 0 0.360 rpy=0 0 0, axis 0 0 -1, limit lower=-3.1415 upper=3.1415 effort=100 velocity=3.4906
- added joint joint_6: type revolute, parent link_5, child link_6, origin xyz=0 0 0 rpy=0 0 0, axis 0 -1 0, limit lower=-1.9198 upper=1.9198 effort=100 velocity=3.4906
- added joint joint_7: type revolute, parent link_6, child link_7, origin xyz=0 0 0.155 rpy=0 0 0, axis 0 0 -1, limit lower=-3.1415 upper=3.1415 effort=100 velocity=6.9813
- added joint link_2-base: type fixed, parent link_2, child base, origin xyz=0 0 0 rpy=0 0 0

Commit message: +Industrial Robots

File: modelos/kr16_2.urdf (robot description, URDF)
Before this commit: robot kuka_kr16_2, 9 links, 8 joints
Links:
- link base_link: mass 2 -> None
- link link_1: mass 2 -> None
- link link_2: mass 2 -> None
- link link_3: mass 2 -> None
- link link_4: mass 2 -> None
- link link_5: mass 2 -> None
- link link_6: mass 2 -> None

File: modelos/kr210l150.urdf (robot description, URDF)
Before this commit: robot kuka_kr210, 9 links, 8 joints
Links:
- link base_link: mass 1572.9 -> None
- link link_1: mass 1385.5 -> None
- link link_2: mass 958.62 -> None
- link link_3: mass 710.03 -> None
- link link_4: mass 173.73 -> None
- link link_5: mass 72.17 -> None
- link link_6: mass 6.3154 -> None

File: modelos/sia10f.urdf (robot description, URDF)
Before this commit: robot motoman_sia10f, 9 links, 8 joints
Joints:
- removed joint link_2-base
- added joint base_link-base: type fixed, parent base_link, child base, origin xyz=0 0 0 rpy=0 0 0
