Commit message: add trail tool0

File: modelos/irb2600.urdf (robot description, URDF)
Before this commit: robot abb_irb2600_12_165, 9 links, 8 joints
Joints:
- joint joint_2: limit lower=-2.705 upper=1.658 effort=0 velocity=3.054 -> lower=-1.658 upper=2.705 effort=0 velocity=3.054

File: modelos/irb6640.urdf (robot description, URDF)
Before this commit: robot abb_irb6640, 11 links, 10 joints
Joints:
- joint joint_cylinder: limit lower=-2.96705973 upper=2.96705973 effort=0 velocity=0 -> (none)
- joint joint_piston: limit lower=0 upper=0.6 effort=0 velocity=0 -> (none)
