Commit message: Add model Puma and Scara arm

File: modelos/cartesian.urdf (robot description, URDF)
Before this commit: robot CartMan, 13 links, 12 joints
Links:
- removed link link_support1
- removed link link_support1x
- removed link link_support1y
- removed link link_support2
- removed link link_support2x
- removed link link_support2y
- removed link link_support3
- removed link link_support4
- added link link_supportz; visual box size=0.07 0.07 1; visual box size=0.07 0.07 1
Joints:
- removed joint base_support1x
- removed joint base_support1y
- removed joint base_support2
- removed joint base_support2x
- removed joint base_support2y
- removed joint base_support3
- removed joint base_support4
- joint base_support1: child link_support1 -> link_supportz; origin xyz=0 0 -0.5 rpy=0 0 0 -> xyz=0 0 0 rpy=0 0 0
- joint joint_3: origin xyz=0 0.12 0 rpy=0 0 0 -> xyz=0 -0.6 0 rpy=0 0 0

File: modelos/katana_robot.urdf (robot description, URDF)
Before this commit: robot katana_450_6m90a, 10 links, 9 joints
Links:
- link katana_gripper_tool_frame: mass 0.0012 -> None
- link katana_l_finger_link: mass 0.0251722230462 -> None
- link katana_r_finger_link: mass 0.0251722230462 -> None
- link link_1: mass 0.74793301875 -> None
- link link_2: mass 0.80174941875 -> None
- link link_3: mass 0.79241664375 -> None
- link link_4: mass 0.69149323125 -> None
- link link_5: mass 0.25622555625 -> None
- link tool0: mass 0.0552136183596 -> None
