Commit message: add + reachability map

File: modelos/sia20d.urdf (robot description, URDF)
Before this commit: robot motoman_sia20d, 10 links, 9 joints
Links:
- removed link link_b
- removed link link_e
- removed link link_l
- removed link link_r
- removed link link_s
- removed link link_t
- removed link link_u
- added link link_1; collision mesh filename=package://rvizglabre/modelos/sia20d/collision/MOTOMAN_AXIS_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; visual mesh filename=package://rvizglabre/modelos/sia20d/visual/MOTOMAN_AXIS_S.s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
- added link link_2; collision mesh filename=package://rvizglabre/modelos/sia20d/collision/MOTOMAN_AXIS_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; visual mesh filename=package://rvizglabre/modelos/sia20d/visual/MOTOMAN_AXIS_L.s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
- added link link_3; collision mesh filename=package://rvizglabre/modelos/sia20d/collision/MOTOMAN_AXIS_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; visual mesh filename=package://rvizglabre/modelos/sia20d/visual/MOTOMAN_AXIS_E.s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
- added link link_4; collision mesh filename=package://rvizglabre/modelos/sia20d/collision/MOTOMAN_AXIS_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; visual mesh filename=package://rvizglabre/modelos/sia20d/visual/MOTOMAN_AXIS_U.s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
- added link link_5; collision mesh filename=package://rvizglabre/modelos/sia20d/collision/MOTOMAN_AXIS_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; visual mesh filename=package://rvizglabre/modelos/sia20d/visual/MOTOMAN_AXIS_R.s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
- added link link_6; collision mesh filename=package://rvizglabre/modelos/sia20d/collision/MOTOMAN_AXIS_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; visual mesh filename=package://rvizglabre/modelos/sia20d/visual/MOTOMAN_AXIS_B.s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
- added link link_7; collision mesh filename=package://rvizglabre/modelos/sia20d/collision/MOTOMAN_AXIS_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; visual mesh filename=package://rvizglabre/modelos/sia20d/visual/MOTOMAN_AXIS_T.s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
Joints:
- removed joint joint_b
- removed joint joint_e
- removed joint joint_l
- removed joint joint_r
- removed joint joint_s
- removed joint joint_t
- removed joint joint_u
- removed joint link_t-tool0
- added joint joint_1: type revolute, parent base_link, child link_1, origin xyz=0 0 0.41 rpy=0 0 0, axis 0 0 1, limit lower=-3.1415 upper=3.1415 effort=100 velocity=2.2689
- added joint joint_2: type revolute, parent link_1, child link_2, origin xyz=0 0 0 rpy=0 0 0, axis 0 1 0, limit lower=-1.9198 upper=1.9198 effort=100 velocity=2.2689
- added joint joint_3: type revolute, parent link_2, child link_3, origin xyz=0 0 0.49 rpy=0 0 0, axis 0 0 1, limit lower=-2.9670 upper=2.9670 effort=100 velocity=2.9670
- added joint joint_4: type revolute, parent link_3, child link_4, origin xyz=0 0 0 rpy=0 0 0, axis 0 -1 0, limit lower=-2.2689 upper=2.2689 effort=100 velocity=2.9670
- added joint joint_5: type revolute, parent link_4, child link_5, origin xyz=0 0 0.420 rpy=0 0 0, axis 0 0 -1, limit lower=-3.1415 upper=3.1415 effort=100 velocity=3.4906
- added joint joint_6: type revolute, parent link_5, child link_6, origin xyz=0 0 0 rpy=0 0 0, axis 0 -1 0, limit lower=-1.9198 upper=1.9198 effort=100 velocity=3.4906
- added joint joint_7: type revolute, parent link_6, child link_7, origin xyz=0 0 0.18 rpy=0 0 0, axis 0 0 -1, limit lower=-3.1415 upper=3.1415 effort=100 velocity=6.9813
- added joint joint_tool0: type fixed, parent link_7, child tool0, origin xyz=0 0 0.0 rpy=0 0 -3.1416
- joint link_l-base: parent link_l -> link_1
