Commit message: fix stl and disable boton to run

File: modelos/kr120r2500.urdf (robot description, URDF)
Before this commit: robot kuka_kr120r2500pro, 9 links, 8 joints
Links:
- link base_link: geometry collision mesh filename=package://rvizglabre/modelos/kr120r2500/collision/base_link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; visual mesh filename=package://rvizglabre/modelos/kr120r2500/visual/base_link.stl
- link link_1: geometry collision mesh filename=package://rvizglabre/modelos/kr120r2500/collision/link_1.stl; visual mesh filename=package://rvizglabre/modelos/kr120r2500/visual/link_1.stl
- link link_2: geometry collision mesh filename=package://rvizglabre/modelos/kr120r2500/collision/link_2.stl; visual mesh filename=package://rvizglabre/modelos/kr120r2500/visual/link_2.stl
- link link_3: geometry collision mesh filename=package://rvizglabre/modelos/kr120r2500/collision/link_3.stl; visual mesh filename=package://rvizglabre/modelos/kr120r2500/visual/link_3.stl
- link link_5: geometry collision mesh filename=package://rvizglabre/modelos/kr120r2500/collision/link_5.stl; visual mesh filename=package://rvizglabre/modelos/kr120r2500/visual/link_5.stl

File: modelos/robot2dof.urdf (robot description, URDF)
Before this commit: robot origins, 4 links, 3 joints
Joints:
- removed joint joint_3
- added joint joint_3-tool0: type revolute, parent link_2, child tool0, origin xyz=0.06 0 0.4 rpy=0 -1.57 0, limit lower=-0.1 upper=0.1 effort=0 velocity=0.5

File: modelos/ur5_robot.urdf (robot description, URDF)
Before this commit: robot ur5, 8 links, 7 joints
Links:
- link base_link: mass 4.0 -> None
- link link_1: mass 3.7 -> None
- link link_2: mass 8.393 -> None
- link link_3: mass 2.275 -> None
- link link_4: mass 1.219 -> None
- link link_5: mass 1.219 -> None
- link link_6: mass 0.1879 -> None
- link tool0: mass 0.1 -> None; geometry collision cylinder length=0.2 radius=0.01; visual cylinder length=0.1 radius=0.01
Joints:
- joint joint6-tool0: origin xyz=0.0 0.18 0.0 rpy=1.570796325 0.0 0.0 -> xyz=0.0 0.15 0.0 rpy=1.570796325 0.0 0.0
