Commit message: Change RPY

File: modelos/armUNI.urdf (robot description, URDF)
Before this commit: robot lynxmotion_al5d, 7 links, 6 joints
Joints:
- removed joint gripper
- added joint joint_5: type revolute, parent link_4, child gripper, origin xyz=0.048 0 0 rpy=0 0 0, axis 0 0 1, limit lower=-1.570795 upper=1.570795 effort=0 velocity=6.98
